File: Hardware/Hardware.kicad_sch (KiCad schematic)
At the start: 25 parts, among them J1 USB_C_Receptacle_USB2.0, U1 ESP32-C3FH4AZ, Y1 40MHz 9pF ±10ppm, Y2 32.768kHz 6pF ±20ppm

Commit message: Schematic progress
Parts:
- added C?: 470n, symbol Device:C
- added C? (x3): 1u, symbol Device:C
- added D?: D_Schottky, symbol Device:D_Schottky
- added J?: Conn_01x02, symbol Connector_Generic:Conn_01x02
- added Q?: AO3401A, Package_TO_SOT_SMD:SOT-23, symbol Transistor_FET:AO3401A
- added R? (x3): 10K, symbol Device:R
- added R?: R01 1%, symbol Device:R
- added R?: 1K6, symbol Device:R
- added U?: TP4054, Package_TO_SOT_SMD:SOT-23-5, symbol local:TP4054
- added U?: BQ27441DRZR-G1A, Package_SON:Texas_S-PDSO-N12, symbol Battery_Management:BQ27441DRZR-G1A
- added U?: XC6206PxxxMR, Package_TO_SOT_SMD:SOT-23-3, symbol Regulator_Linear:XC6206PxxxMR
- C11: Label Near VDDA -> Near VDDA_RTC
- C12: Label Near VDDA_RTC -> Near VDDA
Connections:
- net +3V3: now also C?.1, R?.2, U?.2 (VO)
- net GND: now also C?.2, C?.2, C?.2, C?.2, J?.1 (Pin_1), R?.1, R?.1, R?.2, U?.1 (GND), U?.13 (PAD), U?.2 (GND), U?.3 (V_{SS})
- net VBUS: now also C?.1, D?.2 (A), Q?.1 (G), R?.2, U?.4 (VCC)
- new net: R?.2, U?.5 (PROG)
- new net: C?.1, U?.5 (V_{DD})
- new net: R?.1, U?.10 (BIN)
- new net: J?.2 (Pin_2), R?.1, U?.6 (BAT), U?.8 (SRP)
- new net: C?.1, D?.1 (K), Q?.2 (S), U?.3 (VI)
- new net +BATT: Q?.3 (D), R?.2, U?.3 (BAT), U?.7 (SRN)
- new net SCL: U?.2 (SCL)
- new net SDA: U?.1 (SDA)
- new net ~{CHRG}: R?.1, U?.1 (~{CHRG})
- no-connect marks 4 -> 5
Other:
- note added: "3V3 supply"
- note added: "Also considering the BQ27220"
- note added: "Battery charger"
- note added: "Battery fuel gauge"
- note added: "No VBUS, gate pulled low, mosfet on, +BATT powers LDO VBUS present, gate high, osfet off, diode OR, VBUS > +BATT, VBUS powers LDO Vgs = 0 - 3.7 = -3.7 so Rds = ~50mΩ, could do better"
- moved on the sheet: C1, C10, C11, C12, C13, C2, C3, C4, C5, C6, C7, C8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

Commit message: Hardware done and ordered 🤞
Parts:
- removed D?: D_Schottky, symbol Device:D_Schottky
- removed JP1, JP2: Jumper_2_Open, Jumper:SolderJumper-2_P1.3mm_Open_RoundedPad1.0x1.5mm, symbol Jumper:Jumper_2_Open
- removed R?: 10K, symbol Device:R
- added AE1: Antenna_PCB, local:Texas_SWRA117D_2.4GHz_Left, symbol local:Antenna_PCB
- added C19: 3p3, Capacitor_SMD:C_0402_1005Metric, symbol Device:C
- added C20, C21, C22: 10n, Capacitor_SMD:C_0402_1005Metric, symbol Device:C
- added D1: 1N5819WS, Diode_SMD:D_SOD-323, symbol Diode:1N5819WS
- added J3: ST7789 1.54" LCD, local:1.54 ST7789, symbol Connector_Generic:Conn_01x12
- added J4: SIQ-02FVS3, local:SIQ-02FVS3, symbol Connector_Generic:Conn_01x04
- added L2: 2n2, Inductor_SMD:L_0402_1005Metric, symbol Device:L
- added Q2: AO3400A, Package_TO_SOT_SMD:SOT-23, symbol Transistor_FET:AO3400A
- added R11, R12, R13: 10K, Resistor_SMD:R_0402_1005Metric, symbol Device:R
- added R9: 10R, Resistor_SMD:R_0402_1005Metric, symbol Device:R
- C1, C2: footprint (none) -> Capacitor_SMD:C_0402_1005Metric; LCSC (none) -> C1547
- C10, C7, C8, C9: footprint (none) -> Capacitor_SMD:C_0402_1005Metric; LCSC (none) -> C1525
- C11: footprint (none) -> Capacitor_SMD:C_0402_1005Metric; LCSC (none) -> C52923; Label Near VDDA_RTC -> Near VDDA
- C12: footprint (none) -> Capacitor_SMD:C_0402_1005Metric; LCSC (none) -> C15195
- C13: value 1u -> 3p3; footprint (none) -> Capacitor_SMD:C_0402_1005Metric; LCSC (none) -> C1565
- C14: renamed from C?; footprint (none) -> Capacitor_SMD:C_0402_1005Metric; LCSC (none) -> C47339
- C15, C16, C17: renamed from C?; footprint (none) -> Capacitor_SMD:C_0402_1005Metric; LCSC (none) -> C52923
- C3, C4: footprint (none) -> Capacitor_SMD:C_0402_1005Metric; LCSC (none) -> C1576
- C5: footprint (none) -> Capacitor_SMD:C_0402_1005Metric; LCSC (none) -> C15525
- C6: footprint (none) -> Capacitor_SMD:C_0402_1005Metric; LCSC (none) -> C52923
- J1: LCSC (none) -> C2765186
- J2: renamed from J?; value Conn_01x02 -> Battery; footprint (none) -> Connector_JST:JST_PH_S2B-PH-SM4-TB_1x02-1MP_P2.00mm_Horizontal; LCSC (none) -> C295747
- L1: value 2n >500mA -> 2n2; footprint (none) -> Inductor_SMD:L_0402_1005Metric; LCSC (none) -> C86061
- Q1: renamed from Q?; LCSC (none) -> C15127
- R1, R5: footprint (none) -> Resistor_SMD:R_0402_1005Metric; LCSC (none) -> C25744
- R10, R7: renamed from R?; footprint (none) -> Resistor_SMD:R_0402_1005Metric; LCSC (none) -> C25744
- R2: footprint (none) -> Resistor_SMD:R_0402_1005Metric; LCSC (none) -> C25092
- R3, R4: footprint (none) -> Resistor_SMD:R_0402_1005Metric; LCSC (none) -> C25905
- R6: renamed from R?; footprint (none) -> Resistor_SMD:R_0805_2012Metric; LCSC (none) -> C3024467
- R8: renamed from R?; value 1K6 -> 2K2; footprint (none) -> Resistor_SMD:R_0402_1005Metric; LCSC (none) -> C25879
- U1: LCSC (none) -> C2858491
- U2: renamed from U?; LCSC (none) -> C473397
- U3: renamed from U?; LCSC (none) -> C32574
- U4: renamed from U?; LCSC (none) -> C5446
- Y1: LCSC (none) -> C557159
- Y2: LCSC (none) -> C32346
Connections:
- net +3V3: now also J3.3 (Pin_3), J3.4 (Pin_4)
- net GND: now also J1.S1 (SHIELD), AE1.2 (PCB_Trace), C19.2, C20.2, C21.2, C22.2, J3.1 (Pin_1), J3.12 (Pin_12), J3.5 (Pin_5), J3.6 (Pin_6), J4.3 (Pin_3), Q2.2 (S)
- net MOSI: now also U1.8 (ADC1_CH3/IO3), J3.10 (Pin_10)
- net SCK: now also U1.9 (MTMS/ADC1_CH4/IO4), J3.9 (Pin_9)
- net SCL: now also U1.27 (U0RXD/IO20)
- net SDA: now also U1.28 (U0TXD/IO21)
- net VBUS: now also D1.2 (A)
- net at C16.1, Q1.2 (S), U4.3 (VI): now also D1.1 (K)
- net LNA_IN: now reaches U1.1 (LNA_IN)
- net LNA_IN: now also C13.1, L2.1
- net LCD_CS: now reaches U1.10 (MTDI/ADC2_CH20/IO5)
- net LCD_CS: now also J3.8 (Pin_8)
- net LCD_BL: now reaches U1.12 (MTCK/IO6)
- net LCD_BL: now also Q2.1 (G)
- net LCD_DC: now reaches U1.13 (MTDO/IO7)
- net LCD_DC: now also J3.7 (Pin_7)
- net ENC_B: now reaches U1.14 (IO8)
- net ENC_B: now also C22.1, R13.1
- net ENC_A: now reaches U1.16 (IO10)
- net ENC_A: now also C20.1, R11.1
- net BOOT renamed ENC_SW
- net ENC_SW: now also C21.1, R12.1; no longer C13.1
- net RESET renamed ~{RESET}
- net ~{RESET}: now also J3.11 (Pin_11)
- net ~{CHRG}: no longer names the net of U3.1 (~{CHRG})
- new net: AE1.1 (FEED), C19.1, L2.2
- new net: J4.1 (Pin_1), R11.2
- new net: J4.2 (Pin_2), R12.2
- new net: J4.4 (Pin_4), R13.2
- new net: Q2.3 (D), R9.2
- new net LCD_BL_K: J3.2 (Pin_2), R9.1
- no-connect marks 5 -> 6
Other:
- note added: "Battery charger 450mA charge current"
- note added: "ENC_SW is connected to boot mode pin hence pullup All other inputs will just use built-in pullups on ESP32"
- note added: "GND"
- note added: "LCD_BL_A"
- note added: "No VBUS -> gate pulled low -> mosfet on -> +BATT powers LDO VBUS present -> gate high -> mosfet off -> VBUS > +BATT -> VBUS powers LDO Vgs = 0 - 3.7 = -3.7 so Rds = ~50mΩ, could do better"
- note added: "Only 2mW dissipated"
- note added: "VCC"
- note added: "Z = (35+10j)R"
- note added: "Z = 50R"
- note removed: "Battery charger"
- note removed: "No VBUS, gate pulled low, mosfet on, +BATT powers LDO VBUS present, gate high, osfet off, diode OR, VBUS > +BATT, VBUS powers LDO Vgs = 0 - 3.7 = -3.7 so Rds = ~50mΩ, could do better"
- moved on the sheet: C1, C10, C11, C12, C2, C3, C4, C5, C7, C8, C9, J2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
