File: V2/Hardware/Hardware.kicad_pcb (KiCad board)
At the start: 2 copper layers, 15 parts, among them J1 USB_C_Receptacle_USB2.0, J2 1.54 E-INK, Q1 AO3401A, U1 nRF52840, U2 MCP1700x-180xxTT, Y1 32MHz 8pF ±10ppm, Y2 32.768kHz 6pF ±20ppm

Commit message: Schematic progress
Parts:
- added D2: 1N5819WS, Diode_SMD:D_SOD-323, B.Cu at (131.3, 92.8)
- added D3: 1N5819WS, Diode_SMD:D_SOD-323, B.Cu at (131.3, 95.7)
- added D4: 1N5819WS, Diode_SMD:D_SOD-323, B.Cu at (131.3, 98.7)
- added JP1: Jumper_2_Open, Jumper:SolderJumper-2_P1.3mm_Open_RoundedPad1.0x1.5mm, B.Cu at (124.1, 93.1)
- added Q2: AO3400A, Package_TO_SOT_SMD:SOT-23, B.Cu at (126.7, 99.5)
- added R4: 100K, Resistor_SMD:R_0402_1005Metric, B.Cu at (127.7, 92.3)
- added R5: 10K, Resistor_SMD:R_0402_1005Metric, B.Cu at (127.7, 94.3)
- added R6: 0R47, Resistor_SMD:R_0402_1005Metric, B.Cu at (127.7, 96.3)
- C16, C17, C2, C3, D1, Q1, R1, R2, R3, U2, Y1, Y2: moved to B.Cu
- moved C16 22.2 mm to (141.0, 104.1), turned to 180 degrees
- moved C17 22.2 mm to (141.0, 106.0), turned to 180 degrees
- moved C2 22.2 mm to (141.0, 100.1), turned to 180 degrees
- moved C3 22.2 mm to (141.0, 102.1), turned to 180 degrees
- moved Y1 21.2 mm to (140.5, 115.2), turned to 180 degrees
- moved D1 20.7 mm to (140.2, 111.8), turned to 180 degrees
- moved Q1 20.1 mm to (140.0, 83.8), turned to 180 degrees
- moved U2 20.1 mm to (140.0, 88.2), turned to 180 degrees
- moved Y2 20.0 mm to (139.9, 108.7), turned to 180 degrees
- moved R1 16.4 mm to (138.1, 100.1), turned to 180 degrees
- moved R2 16.4 mm to (138.1, 102.1), turned to 180 degrees
- moved R3 16.4 mm to (138.1, 104.1), turned to 180 degrees
- turned U1 to 45 degrees
Connections:
- J2 pad 10: unconnected-(J2-Pin_10-Pad10) -> /EINK_RES
- J2 pad 11: unconnected-(J2-Pin_11-Pad11) -> /EINK_DC
- J2 pad 12: unconnected-(J2-Pin_12-Pad12) -> /EINK_CS
- J2 pad 13: unconnected-(J2-Pin_13-Pad13) -> /EINK_SCLK
- J2 pad 14: unconnected-(J2-Pin_14-Pad14) -> /EINK_SDI
- J2 pad 15: unconnected-(J2-Pin_15-Pad15) -> +1V8
- J2 pad 16: unconnected-(J2-Pin_16-Pad16) -> +1V8
- J2 pad 17: unconnected-(J2-Pin_17-Pad17) -> GND
- J2 pad 18: unconnected-(J2-Pin_18-Pad18) -> Net-(J2-Pin_18)
- J2 pad 19: unconnected-(J2-Pin_19-Pad19) -> Net-(J2-Pin_19)
- J2 pad 2: unconnected-(J2-Pin_2-Pad2) -> /GDR
- J2 pad 20: unconnected-(J2-Pin_20-Pad20) -> Net-(J2-Pin_20)
- J2 pad 21: unconnected-(J2-Pin_21-Pad21) -> /PREVGH
- J2 pad 22: unconnected-(J2-Pin_22-Pad22) -> Net-(J2-Pin_22)
- J2 pad 23: unconnected-(J2-Pin_23-Pad23) -> /PREVGL
- J2 pad 24: unconnected-(J2-Pin_24-Pad24) -> Net-(J2-Pin_24)
- J2 pad 3: unconnected-(J2-Pin_3-Pad3) -> /RESE
- J2 pad 4: unconnected-(J2-Pin_4-Pad4) -> Net-(J2-Pin_4)
- J2 pad 5: unconnected-(J2-Pin_5-Pad5) -> Net-(J2-Pin_5)
- J2 pad 8: unconnected-(J2-Pin_8-Pad8) -> GND
- J2 pad 9: unconnected-(J2-Pin_9-Pad9) -> /EINK_BUSY
- U1 pad A10: unconnected-(U1-AIN5/P0.29-PadA10) -> /EINK_SDI
- U1 pad A8: unconnected-(U1-AIN7/P0.31-PadA8) -> /EINK_SCLK
- U1 pad AC13: unconnected-(U1-P0.18/~{RESET}-PadAC13) -> /~{RESET}
- U1 pad B11: unconnected-(U1-AIN4/P0.28-PadB11) -> /EINK_DC
- U1 pad B9: unconnected-(U1-AIN6/P0.30-PadB9) -> /EINK_CS
- U1 pad G1: unconnected-(U1-P0.26-PadG1) -> /EINK_RES
- U1 pad H2: unconnected-(U1-P0.27-PadH2) -> /EINK_BUSY
