File: V2/Hardware/Hardware.kicad_sch (KiCad schematic)
At the start: 33 parts, among them J1 USB_C_Receptacle_USB2.0, J2 1.54 E-INK, Q1 AO3401A, U1 nRF52840, U2 MCP1700x-180xxTT, Y1 32MHz 8pF ±10ppm, Y2 32.768kHz 6pF ±20ppm

Commit message: Schematic progress
Parts:
- added C19, C20, C21, C22, C24, C25, C28, C29: 4u7, symbol Device:C
- added C23, C26, C27, C30: 1u, symbol Device:C
- added D2, D3, D4: 1N5819WS, Diode_SMD:D_SOD-323, symbol Diode:1N5819WS
- added JP1: Jumper_2_Open, Jumper:SolderJumper-2_P1.3mm_Open_RoundedPad1.0x1.5mm, symbol Jumper:Jumper_2_Open
- added Q2: AO3400A, Package_TO_SOT_SMD:SOT-23, symbol Transistor_FET:AO3400A
- added R8: 10K, Resistor_SMD:R_0402_1005Metric, symbol Device:R
- added R8: 0R47, Resistor_SMD:R_0402_1005Metric, symbol Device:R
- added R8: 100K, Resistor_SMD:R_0402_1005Metric, symbol Device:R
- L2: value 15n -> 10u
Connections:
- net +1V8: now also J2.15 (Pin_15), J2.16 (Pin_16), L2.1, C19.1, C26.1, R8.2
- net GND: now also J2.17 (Pin_17), J2.8 (Pin_8), C19.2, C21.2, C22.2, C23.2, C24.2, C25.2, C26.2, C27.2, C28.2, C29.2, C30.2, D3.1 (K), JP1.1 (A), R8.1, R8.1
- net at C1.1, C4.1, U1.B5 (DEC4)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: now also L3.1; no longer L2.1
- net at L2.2: now also C20.1, D4.2 (A), Q2.3 (D); no longer L3.1
- net EINK_SDI: now reaches U1.A10 (AIN5/P0.29)
- net EINK_SDI: now also J2.14 (Pin_14)
- net EINK_SCLK: now reaches U1.A8 (AIN7/P0.31)
- net EINK_SCLK: now also J2.13 (Pin_13)
- net ~{RESET}: now reaches U1.AC13 (P0.18/~{RESET})
- net ~{RESET}: now also JP1.2 (B), R8.1
- net EINK_DC: now reaches U1.B11 (AIN4/P0.28)
- net EINK_DC: now also J2.11 (Pin_11)
- net EINK_CS: now reaches U1.B9 (AIN6/P0.30)
- net EINK_CS: now also J2.12 (Pin_12)
- net EINK_RES: now reaches U1.G1 (P0.26)
- net EINK_RES: now also J2.10 (Pin_10)
- net EINK_BUSY: now reaches U1.H2 (P0.27)
- net EINK_BUSY: now also J2.9 (Pin_9)
- net at J2.18 (Pin_18): now also C27.1
- net at J2.19 (Pin_19): now also C23.1
- net GDR: now reaches J2.2 (Pin_2)
- net GDR: now also Q2.1 (G), R8.2
- net at J2.20 (Pin_20): now also C28.1
- net PREVGH: now reaches J2.21 (Pin_21)
- net PREVGH: now also C21.1, D4.1 (K)
- net at J2.22 (Pin_22): now also C29.1
- net PREVGL: now reaches J2.23 (Pin_23)
- net PREVGL: now also C24.1, D2.2 (A)
- net at J2.24 (Pin_24): now also C30.1
- net RESE: now reaches J2.3 (Pin_3)
- net RESE: now also Q2.2 (S), R8.2
- net at J2.4 (Pin_4): now also C22.1
- net at J2.5 (Pin_5): now also C25.1
- new net: C20.2, D2.1 (K), D3.2 (A)
- no-connect marks 4 -> 7
Other:
- moved on the sheet: AE1, C1, C10, C11, C12, C13, C14, C15, C18, C2, C3, C4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
