File: V1/Hardware/Hardware.kicad_sch (KiCad schematic)
At the start: 50 parts, among them J1 USB_C_Receptacle_USB2.0, J2 Battery, J3 ST7789 1.54" LCD, J4 SIQ-02FVS3, Q1 AO3401A, Q2 AO3400A, U1 ESP32-C3FH4AZ, U2 BQ27441DRZR-G1A, U3 TP4054, U4 XC6206PxxxMR, Y1 40MHz 9pF ±10ppm, Y2 32.768kHz 6pF ±20ppm

Commit message: Update V1 schematic to e-ink
Parts:
- removed J3: ST7789 1.54" LCD, local:1.54 ST7789, symbol Connector_Generic:Conn_01x12
- removed R9: 10R, Resistor_SMD:R_0402_1005Metric, symbol Device:R
- added C18, C23, C24, C25, C27, C28, C31, C32: 4u7, symbol Device:C
- added C26, C29, C30, C33: 1u, symbol Device:C
- added D2, D3, D4: 1N5819WS, Diode_SMD:D_SOD-323, symbol Diode:1N5819WS
- added J3: 1.54 E-INK, local:1.54_Epaper_Display, symbol Connector_Generic:Conn_01x24
- added L3: 68u, symbol Device:L
- added R8: 10K, Resistor_SMD:R_0402_1005Metric, symbol Device:R
- added R8: 2R2, Resistor_SMD:R_0402_1005Metric, symbol Device:R
- added SW?: SW_Push, symbol Switch:SW_Push
- Q2: LCSC C20917 -> (none)
Connections:
- net +3V3: now also C18.1, C29.1, J3.15 (Pin_15), J3.16 (Pin_16), L3.1
- net GND: now also C18.2, C24.2, C25.2, C26.2, C27.2, C28.2, C29.2, C30.2, C31.2, C32.2, C33.2, D3.1 (K), J3.17 (Pin_17), J3.8 (Pin_8), R8.1, R8.1; no longer Q2.2 (S)
- net at Q2.3 (D): now also C23.1, D4.2 (A), L3.2
- net EINK_RES: now reaches U1.6 (ADC1_CH2/IO2)
- net EINK_RES: now also J3.10 (Pin_10)
- net LCD_BL renamed EINK_BUSY
- net EINK_BUSY: now also J3.9 (Pin_9); no longer Q2.1 (G)
- net LCD_CS renamed EINK_CS
- net EINK_CS: now also J3.12 (Pin_12)
- net LCD_DC renamed EINK_DC
- net EINK_DC: now also J3.11 (Pin_11)
- net MOSI renamed EINK_SDI
- net EINK_SDI: now also J3.14 (Pin_14)
- net SCK renamed EINK_SCLK
- net EINK_SCLK: now also J3.13 (Pin_13)
- new net: C26.1, J3.19 (Pin_19)
- new net: C28.1, J3.5 (Pin_5)
- new net: C32.1, J3.22 (Pin_22)
- new net: C23.2, D2.1 (K), D3.2 (A)
- new net: C31.1, J3.20 (Pin_20)
- new net: C25.1, J3.4 (Pin_4)
- new net: C30.1, J3.18 (Pin_18)
- new net: C33.1, J3.24 (Pin_24)
- new net GDR: J3.2 (Pin_2), Q2.1 (G), R8.2
- new net PREVGH: C24.1, D4.1 (K), J3.21 (Pin_21)
- new net PREVGL: C27.1, D2.2 (A), J3.23 (Pin_23)
- new net RESE: J3.3 (Pin_3), Q2.2 (S), R8.2
- no-connect marks 6 -> 8
Other:
- note added: "Potential buttons TP12422663 TS24CA K2-1114SA-A4SW-06"
- note removed: "GND"
- note removed: "LCD_BL_A"
- note removed: "VCC"
