File: NRF52/Hardware/Hardware.kicad_sch (KiCad schematic)
At the start: 53 parts, among them J1 USB_C_Receptacle_USB2.0, J2 1.54 E-INK, Q1 AO3401A, Q2 AO3400A, U1 nRF52840, U2 MCP1700x-180xxTT, Y1 32MHz 8pF ±10ppm, Y2 32.768kHz 6pF ±20ppm

Commit message: Progress on NRF52 version hardware
Parts:
- removed JP1: Jumper_2_Open, Jumper:SolderJumper-2_P1.3mm_Open_RoundedPad1.0x1.5mm, symbol Jumper:Jumper_2_Open
- removed U2: MCP1700x-180xxTT, Package_TO_SOT_SMD:SOT-23, symbol Regulator_Linear:MCP1700x-180xxTT
- added C14: 470n, Capacitor_SMD:C_0603_1608Metric, symbol Device:C
- added C15, C34, C35, C36, C37: 1u, Capacitor_SMD:C_0402_1005Metric, symbol Device:C
- added C33: 100n, Capacitor_SMD:C_0402_1005Metric, symbol Device:C
- added D2 (x2): 1N5819WS, Diode_SMD:D_SOD-323, symbol Diode:1N5819WS
- added J2: Battery, local:Battery Pads, symbol Connector_Generic:Conn_01x02
- added J3: Conn_01x04, local:Program_Pads, symbol Connector_Generic:Conn_01x04
- added Q1: AO3401A, Package_TO_SOT_SMD:SOT-23, symbol Transistor_FET:AO3401A
- added Q3: AO3400A, Package_TO_SOT_SMD:SOT-23, symbol Transistor_FET:AO3400A
- added R6: R01 1%, Resistor_SMD:R_0805_2012Metric, symbol Device:R
- added R7 (x3), R8 (x2): 10K, Resistor_SMD:R_0402_1005Metric, symbol Device:R
- added R8: 2K2, Resistor_SMD:R_0402_1005Metric, symbol Device:R
- added R8: 1M, Resistor_SMD:R_0402_1005Metric, symbol Device:R
- added R8: 100K, Resistor_SMD:R_0402_1005Metric, symbol Device:R
- added SW1, SW2, SW3: SW_Push, Button_Switch_SMD:Panasonic_EVQPUL_EVQPUC, symbol Switch:SW_Push
- added U2: BQ27441DRZR-G1A, Package_SON:Texas_S-PDSO-N12, symbol Battery_Management:BQ27441DRZR-G1A
- added U3: TP4054, Package_TO_SOT_SMD:SOT-23-5, symbol local:TP4054
- added U4: XC6206PxxxMR, Package_TO_SOT_SMD:SOT-23-3, symbol Regulator_Linear:XC6206PxxxMR
- added U5: LSM6DS3, Package_LGA:LGA-14_3x2.5mm_P0.5mm_LayoutBorder3x4y, symbol Sensor_Motion:LSM6DS3
- added U6: DS3231MZ, Package_SO:SOIC-8_3.9x4.9mm_P1.27mm, symbol Timer_RTC:DS3231MZ
- AE1: footprint (none) -> RF_Antenna:Texas_SWRA117D_2.4GHz_Right
- C1, C12, C23, C26, C27, C30: footprint (none) -> Capacitor_SMD:C_0402_1005Metric; LCSC (none) -> C52923
- C10, C11, C13, C19, C20, C21, C22, C24, C25, C28, C29: footprint (none) -> Capacitor_SMD:C_0402_1005Metric; LCSC (none) -> C23733
- C14, C15, C18, C8: footprint (none) -> Capacitor_SMD:C_0402_1005Metric; LCSC (none) -> C1525
- C4: footprint (none) -> Capacitor_SMD:C_0603_1608Metric; LCSC (none) -> C1622
- C5: footprint (none) -> Capacitor_SMD:C_0402_1005Metric; LCSC (none) -> C296004
- C6: footprint (none) -> Capacitor_SMD:C_0402_1005Metric; LCSC (none) -> C301959
- C7: footprint (none) -> Capacitor_SMD:C_0402_1005Metric; LCSC (none) -> C1546
- C9: footprint (none) -> Capacitor_SMD:C_0402_1005Metric; LCSC (none) -> C172820
- D2, D3, D4: LCSC (none) -> C191023
- J1: LCSC (none) -> C2765186
- J2: LCSC (none) -> C2911766
- L1: footprint (none) -> Inductor_SMD:L_0402_1005Metric; LCSC (none) -> C395070
- L2: footprint (none) -> Inductor_SMD:L_0603_1608Metric; LCSC (none) -> C1035
- L3: footprint (none) -> Inductor_SMD:L_0603_1608Metric; LCSC (none) -> C57838
- Q2: LCSC (none) -> C20917
- R1, R2: LCSC (none) -> C100665
- R8: value 100K -> 10K
- U1: LCSC (none) -> C190794
Connections:
- net +BATT: now also C33.1, Q1.2 (S), R6.2, R8.2, U2.7 (SRN), U3.3 (BAT); no longer Q1.3 (D)
- net EINK_BUSY: now also U1.U1 (TRACEDATA1/P0.12); no longer U1.H2 (P0.27)
- net EINK_CS: now also U1.L1 (P0.06); no longer U1.B9 (AIN6/P0.30)
- net EINK_DC: now also U1.B17 (P1.12), U1.N1 (P0.08); no longer U1.B11 (AIN4/P0.28)
- net EINK_RES: now also U1.R1 (TRACEDATA3/P1.09); no longer U1.G1 (P0.26)
- net EINK_SCLK: now also U1.J1 (AIN2/P0.04); no longer U1.A8 (AIN7/P0.31)
- net EINK_SDI: now also U1.G1 (P0.26); no longer U1.A10 (AIN5/P0.29)
- net GND: now also C14.2, C15.2, C34.1, C35.2, C36.2, C37.2, J2.1 (Pin_1), J3.1 (Pin_1), Q3.2 (S), R7.2, R8.1, R8.1, R8.1, SW1.1, SW2.2, SW3.2, U2.13 (PAD), U2.3 (V_{SS}), U3.2 (GND), U4.1 (GND), U5.1 (SDO/SA0), U5.2 (SDX), U5.3 (SCX), U5.6 (GND), U5.7 (GND), U6.2 (VCC), U6.5 (GND)
- net VBUS: now also C15.1, R8.2, U3.4 (VCC)
- net ~{RESET}: now also J3.4 (Pin_4)
- net at D2.1 (K), Q1.2 (S): now also C34.2, U4.3 (VI)
- net SWDCLK: now reaches U1.AA24 (SWDCLK)
- net SWDCLK: now also J3.3 (Pin_3)
- net POWER_LATCH: now reaches U1.AC11 (P0.16)
- net POWER_LATCH: now also Q3.1 (G), R8.2
- net SWDIO: now reaches U1.AC24 (SWDIO)
- net SWDIO: now also J3.2 (Pin_2)
- net DOWN_BUTTON: now reaches U1.AC9 (P0.14)
- net DOWN_BUTTON: now also SW3.1
- net POWER_BUTTON: now reaches U1.AD10 (P0.15)
- net POWER_BUTTON: now also D2.2 (A)
- net VBUS_PRESENT: now reaches U1.AD12 (P0.17)
- net VBUS_PRESENT: now also R8.1, R8.2
- net RTC_INT: now reaches U1.AD16 (P0.20)
- net RTC_INT: now also U1.M2 (TRACECLK/P0.07), U6.3 (~{INT}/SQW)
- net IMU_INT: now reaches U1.AD18 (P0.22)
- net IMU_INT: now also U5.4 (INT1)
- net SDA: now reaches U1.AD20 (P0.24)
- net SDA: now also R7.2, U2.1 (SDA), U5.14 (SDA), U6.8 (SCL)
- net SCL: now reaches U1.AD22 (TRACEDATA0/P1.00)
- net SCL: now also R7.2, U2.2 (SCL), U5.13 (SCL), U6.7 (SDA)
- net UP_BUTTON: now reaches U1.AD8 (P0.13)
- net UP_BUTTON: now also SW2.1
- net +1V8 renamed +3V3
- net +3V3: now also C35.1, C36.1, C37.1, R7.1, R7.1, U4.2 (VO), U5.12 (CS), U5.5 (VDDIO), U5.8 (VDD), U6.6 (VBAT)
- new net: C33.2, D2.2 (A), Q1.1 (G), Q3.3 (D), R8.1
- new net: Q1.3 (D), Q1.3 (D)
- new net: R7.1, U2.10 (BIN)
- new net: C14.1, U2.5 (V_{DD})
- new net: J2.2 (Pin_2), R6.1, U2.6 (BAT), U2.8 (SRP)
- new net: D2.1 (K), D2.1 (K), SW1.2
- new net: R8.2, U3.5 (PROG)
- no-connect marks 7 -> 36
Other:
- note added: "Also considering the BQ27220"
- note added: "Battery charger 450mA charge current"
- note added: "Battery fuel gauge"
- note added: "Only 2mW dissipated"
- note added: "~3.5V dropout 200mA max Wanted to use 1.8V but not sure how eink would react"
- note removed: "2.3-6.0V 200mA max 1.6uA quiescent"
- moved on the sheet: AE1, C1, C10, C11, C12, C13, C14, C15, C18, C19, C2, C20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

Commit message: Correct e-ink driver components
Parts:
- C20, C21, C22, C24, C25, C28, C29: footprint Capacitor_SMD:C_0402_1005Metric -> Capacitor_SMD:C_0805_2012Metric; LCSC C23733 -> C98192
- C23, C26, C27, C30: footprint Capacitor_SMD:C_0402_1005Metric -> Capacitor_SMD:C_0603_1608Metric; LCSC C52923 -> C15849
- L2: footprint Inductor_SMD:L_0603_1608Metric -> Inductor_SMD:L_Taiyo-Yuden_MD-3030; LCSC C1035 -> C497541
Changed lines of the file:
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@@
       (effects (font (size 1.27 1.27)) (justify right))
     )
-    (property "Footprint" "Capacitor_SMD:C_0402_1005Metric" (at 438.15 309.5752 0)
+    (property "Footprint" "Capacitor_SMD:C_0805_2012Metric" (at 438.15 309.5752 0)
       (effects (font (size 1.27 1.27)) hide)
     )
@@
       (effects (font (size 1.27 1.27)) hide)
     )
-    (property "LCSC" "C23733" (at 441.96 308.61 0)
+    (property "LCSC" "C98192" (at 441.96 308.61 0)
       (effects (font (size 1.27 1.27)) hide)
     )
@@
       (effects (font (size 1.27 1.27)) (justify right))
     )
-    (property "Footprint" "Capacitor_SMD:C_0402_1005Metric" (at 438.15 299.4152 0)
+    (property "Footprint" "Capacitor_SMD:C_0603_1608Metric" (at 438.15 299.4152 0)
       (effects (font (size 1.27 1.27)) hide)
     )
@@
       (effects (font (size 1.27 1.27)) hide)
     )
-    (property "LCSC" "C52923" (at 441.96 298.45 0)
+    (property "LCSC" "C15849" (at 441.96 298.45 0)
       (effects (font (size 1.27 1.27)) hide)
     )
@@
       (effects (font (size 1.27 1.27)))
     )
-    (property "Footprint" "Inductor_SMD:L_0603_1608Metric" (at 365.76 289.56 0)
+    (property "Footprint" "Inductor_SMD:L_Taiyo-Yuden_MD-3030" (at 365.76 289.56 0)
       (effects (font (size 1.27 1.27)) hide)
     )
@@
       (effects (font (size 1.27 1.27)) hide)
     )
-    (property "LCSC" "C1035" (at 365.76 289.56 0)
+    (property "LCSC" "C497541" (at 365.76 289.56 0)
       (effects (font (size 1.27 1.27)) hide)
     )
@@
       (effects (font (size 1.27 1.27)) (justify right))
     )
-    (property "Footprint" "Capacitor_SMD:C_0402_1005Metric" (at 430.53 317.1952 0)
+    (property "Footprint" "Capacitor_SMD:C_0805_2012Metric" (at 430.53 317.1952 0)
       (effects (font (size 1.27 1.27)) hide)
     )
@@
       (effects (font (size 1.27 1.27)) hide)
     )
-    (property "LCSC" "C23733" (at 434.34 316.23 0)
+    (property "LCSC" "C98192" (at 434.34 316.23 0)
       (effects (font (size 1.27 1.27)) hide)
     )
@@
       (effects (font (size 1.27 1.27)) (justify right))
     )
-    (property "Footprint" "Capacitor_SMD:C_0402_1005Metric" (at 438.15 304.4952 0)
+    (property "Footprint" "Capacitor_SMD:C_0603_1608Metric" (at 438.15 304.4952 0)
       (effects (font (size 1.27 1.27)) hide)
     )
@@
       (effects (font (size 1.27 1.27)) hide)
     )
-    (property "LCSC" "C52923" (at 441.96 303.53 0)
+    (property "LCSC" "C15849" (at 441.96 303.53 0)
       (effects (font (size 1.27 1.27)) hide)
     )
@@
       (effects (font (size 1.27 1.27)) (justify right))
     )
-    (property "Footprint" "Capacitor_SMD:C_0402_1005Metric" (at 430.53 268.9352 0)
+    (property "Footprint" "Capacitor_SMD:C_0805_2012Metric" (at 430.53 268.9352 0)
       (effects (font (size 1.27 1.27)) hide)
     )
@@
       (effects (font (size 1.27 1.27)) hide)
     )
-    (property "LCSC" "C23733" (at 434.34 267.97 0)
+    (property "LCSC" "C98192" (at 434.34 267.97 0)
       (effects (font (size 1.27 1.27)) hide)
     )
@@
       (effects (font (size 1.27 1.27)) (justify right))
     )
-    (property "Footprint" "Capacitor_SMD:C_0402_1005Metric" (at 438.15 271.4752 0)
+    (property "Footprint" "Capacitor_SMD:C_0805_2012Metric" (at 438.15 271.4752 0)
       (effects (font (size 1.27 1.27)) hide)
     )
@@
       (effects (font (size 1.27 1.27)) hide)
     )
-    (property "LCSC" "C23733" (at 441.96 270.51 0)
+    (property "LCSC" "C98192" (at 441.96 270.51 0)
       (effects (font (size 1.27 1.27)) hide)
     )
@@
       (effects (font (size 1.27 1.27)) (justify right))
     )
-    (property "Footprint" "Capacitor_SMD:C_0402_1005Metric" (at 438.15 319.7352 0)
+    (property "Footprint" "Capacitor_SMD:C_0603_1608Metric" (at 438.15 319.7352 0)
       (effects (font (size 1.27 1.27)) hide)
     )
@@
       (effects (font (size 1.27 1.27)) hide)
     )
-    (property "LCSC" "C52923" (at 441.96 318.77 0)
+    (property "LCSC" "C15849" (at 441.96 318.77 0)
       (effects (font (size 1.27 1.27)) hide)
     )
@@
       (effects (font (size 1.27 1.27)) (justify right))
     )
-    (property "Footprint" "Capacitor_SMD:C_0402_1005Metric" (at 438.15 314.6552 0)
+    (property "Footprint" "Capacitor_SMD:C_0805_2012Metric" (at 438.15 314.6552 0)
       (effects (font (size 1.27 1.27)) hide)
     )
@@
       (effects (font (size 1.27 1.27)) hide)
     )
-    (property "LCSC" "C23733" (at 441.96 313.69 0)
+    (property "LCSC" "C98192" (at 441.96 313.69 0)
       (effects (font (size 1.27 1.27)) hide)
     )
@@
       (effects (font (size 1.27 1.27)) (justify right))
     )
-    (property "Footprint" "Capacitor_SMD:C_0402_1005Metric" (at 430.53 307.0352 0)
+    (property "Footprint" "Capacitor_SMD:C_0603_1608Metric" (at 430.53 307.0352 0)
       (effects (font (size 1.27 1.27)) hide)
     )
@@
       (effects (font (size 1.27 1.27)) hide)
     )
-    (property "LCSC" "C52923" (at 434.34 306.07 0)
+    (property "LCSC" "C15849" (at 434.34 306.07 0)
       (effects (font (size 1.27 1.27)) hide)
     )
@@
       (effects (font (size 1.27 1.27)) (justify left))
     )
-    (property "Footprint" "Capacitor_SMD:C_0402_1005Metric" (at 392.1252 297.18 0)
+    (property "Footprint" "Capacitor_SMD:C_0805_2012Metric" (at 392.1252 297.18 0)
       (effects (font (size 1.27 1.27)) hide)
     )
@@
       (effects (font (size 1.27 1.27)) hide)
     )
-    (property "LCSC" "C23733" (at 391.16 293.37 0)
+    (property "LCSC" "C98192" (at 391.16 293.37 0)
       (effects (font (size 1.27 1.27)) hide)
     )
@@
       (effects (font (size 1.27 1.27)) (justify left))
     )
-    (property "Footprint" "Capacitor_SMD:C_0402_1005Metric" (at 377.4948 276.86 0)
+    (property "Footprint" "Capacitor_SMD:C_0805_2012Metric" (at 377.4948 276.86 0)
       (effects (font (size 1.27 1.27)) hide)
     )
@@
       (effects (font (size 1.27 1.27)) hide)
     )
-    (property "LCSC" "C23733" (at 378.46 280.67 0)
+    (property "LCSC" "C98192" (at 378.46 280.67 0)
       (effects (font (size 1.27 1.27)) hide)
     )

Commit message: NRF52 hardware as ordered
Parts:
- removed C14: 470n, Capacitor_SMD:C_0603_1608Metric, symbol Device:C
- removed C23, C26, C27, C30: 1u, Capacitor_SMD:C_0603_1608Metric, symbol Device:C
- removed C24, C25, C28, C29: 4u7, Capacitor_SMD:C_0805_2012Metric, symbol Device:C
- removed C33: 100n, Capacitor_SMD:C_0402_1005Metric, symbol Device:C
- removed D2 (x3), D3, D4: 1N5819WS, Diode_SMD:D_SOD-323, symbol Diode:1N5819WS
- removed J2: Battery, local:Battery Pads, symbol Connector_Generic:Conn_01x02
- removed J2: 1.54 E-INK, local:1.54_Epaper_Display, symbol Connector_Generic:Conn_01x24
- removed L2: 10u, Inductor_SMD:L_Taiyo-Yuden_MD-3030, symbol Device:L
- removed Q3: AO3400A, Package_TO_SOT_SMD:SOT-23, symbol Transistor_FET:AO3400A
- removed R6: R01 1%, Resistor_SMD:R_0805_2012Metric, symbol Device:R
- removed R7, R8 (x4): 10K, Resistor_SMD:R_0402_1005Metric, symbol Device:R
- removed R8: 1M, Resistor_SMD:R_0402_1005Metric, symbol Device:R
- removed R8: 0R47, Resistor_SMD:R_0402_1005Metric, symbol Device:R
- removed U2: BQ27441DRZR-G1A, Package_SON:Texas_S-PDSO-N12, symbol Battery_Management:BQ27441DRZR-G1A
- added J2: LCD, Connector_FFC-FPC:Molex_54548-1071_1x10-1MP_P0.5mm_Horizontal, symbol Connector_Generic:Conn_01x10
- added J2: MOTOR, local:Battery Pads, symbol Connector_Generic:Conn_01x02
- added J2: BAT, local:Battery Pads, symbol Connector_Generic:Conn_01x02
- added JP1: SolderJumper_2_Open, Jumper:SolderJumper-2_P1.3mm_Open_TrianglePad1.0x1.5mm, symbol Jumper:SolderJumper_2_Open
- added R7 (x4): 10K, Resistor_SMD:R_0402_1005Metric, symbol Device:R
- added R8 (x2): 100K, Resistor_SMD:R_0402_1005Metric, symbol Device:R
- added TP2: LCD_REFRESH, TestPoint:TestPoint_Pad_D1.0mm, symbol Connector:TestPoint
- added U3: MAX17048, Package_DFN_QFN:TDFN-8-1EP_2x2mm_P0.5mm_EP0.8x1.2mm, symbol local:MAX17048
- added U7: W25Q128JVS, Package_SO:SOIC-8_5.23x5.23mm_P1.27mm, symbol Memory_Flash:W25Q128JVS
- AE1: footprint RF_Antenna:Texas_SWRA117D_2.4GHz_Right -> local:Texas_SWRA117D_2.4GHz_Left
- C19: value 4u7 -> 100n; LCSC C23733 -> C1525
- C20: value 4u7 -> 100p; footprint Capacitor_SMD:C_0805_2012Metric -> Capacitor_SMD:C_0402_1005Metric; LCSC C98192 -> C52923
- C21, C22: value 4u7 -> 1u; footprint Capacitor_SMD:C_0805_2012Metric -> Capacitor_SMD:C_0402_1005Metric; LCSC C98192 -> C52923
- J3: value Conn_01x04 -> PROG
- R8: LCSC C25744 -> C25741
Connections:
- net EINK_CS is gone; now on net DOWN_BUTTON: U1.L1 (P0.06)
- net EINK_SDI is gone; now on net UP_BUTTON: U1.G1 (P0.26)
- net GDR is gone; now on net MOTOR_EN: Q2.1 (G)
- net PREVGH is gone; now on net +3V3: C21.1
- net RESE is gone; now on net GND: Q2.2 (S)
- net VBUS_PRESENT is gone; now on net ~{RESET}: U1.AD12 (P0.17)
- net +3V3: now also C20.1, C22.1, J2.2 (Pin_2), J2.5 (Pin_5), J2.6 (Pin_6), J2.7 (Pin_7), J2.8 (Pin_8), R7.1, R7.1, R7.1, R7.1, R8.1, U7.8 (VCC); no longer C19.1
- net +BATT: now also C19.1, Q1.3 (D), Q1.3 (D), JP1.2 (B), U3.2 (CELL), U3.3 (VDD); no longer Q1.2 (S), R8.2, U3.3 (BAT)
- net DOWN_BUTTON: no longer U1.AC9 (P0.14)
- net GND: now also C20.2, SW1.2, J2.1 (Pin_1), J2.10 (Pin_10), J2.9 (Pin_9), R8.2, U3.1 (CTG), U3.4 (GND), U3.6 (QSTRT), U3.9 (GND), U7.4 (GND); no longer SW1.1, U6.2 (VCC)
- net IMU_INT: now also U1.W24 (P1.02); no longer U1.AD18 (P0.22)
- net POWER_LATCH: now also Q1.1 (G), R8.1, U1.N1 (P0.08); no longer U1.AC11 (P0.16)
- net SWDCLK: now also J3.2 (Pin_2); no longer J3.3 (Pin_3)
- net SWDIO: now also J3.3 (Pin_3); no longer J3.2 (Pin_2)
- net UP_BUTTON: no longer U1.AD8 (P0.13)
- net at Q2.3 (D): now also J2.1 (Pin_1); no longer C20.1
- net LCD_SDI: now reaches U1.A10 (AIN5/P0.29)
- net LCD_SDI: now also J2.2 (Pin_2)
- net LCD_SCLK: now reaches U1.A12 (AIN0/P0.02)
- net LCD_SCLK: now also J2.1 (Pin_1)
- net RTC_SDA: now reaches U1.A14 (P1.15)
- net RTC_SDA: now also R7.2, U6.8 (SCL)
- net RTC_SCL: now reaches U1.A16 (P1.13)
- net RTC_SCL: now also R7.2, U6.7 (SDA)
- net MOTOR_EN: now reaches U1.A20 (P1.10)
- net MOTOR_EN: now also R8.1
- net LCD_CS: now reaches U1.A8 (AIN7/P0.31)
- net LCD_CS: now also J2.3 (Pin_3)
- net QSPI_D3: now reaches U1.J24 (NFC2/P0.10)
- net QSPI_D3: now also U7.7 (IO3)
- net QSPI_SCK: now reaches U1.R24 (P1.06)
- net QSPI_SCK: now also U7.6 (CLK)
- net QSPI_D0: now reaches U1.U24 (P1.04)
- net QSPI_D0: now also U7.5 (DI(IO0))
- net EINK_BUSY renamed FG_SCL
- net FG_SCL: now also R7.2, U3.7 (SCL)
- net EINK_DC: no longer names the net of U1.B17 (P1.12)
- net EINK_DC: no longer U1.N1 (P0.08)
- net EINK_RES renamed FG_SDA
- net FG_SDA: now also R7.2, U3.8 (SDA)
- net EINK_SCLK renamed MENU_BUTTON
- net MENU_BUTTON: now also SW1.1
- net POWER_BUTTON renamed IMU_SCL
- net IMU_SCL: now also U5.13 (SCL), R7.2
- removed net RTC_INT: U1.AD16 (P0.20), U1.M2 (TRACECLK/P0.07), U6.3 (~{INT}/SQW)
- removed net SCL: R7.2, U1.AD22 (TRACEDATA0/P1.00), U5.13 (SCL), U6.7 (SDA)
- removed net SDA: R7.2, U1.AD20 (P0.24), U5.14 (SDA), U6.8 (SCL)
- new net: J2.2 (Pin_2), JP1.1 (A), Q1.2 (S), R8.2, U3.3 (BAT)
- new net IMU_SDA: R7.2, U1.AD8 (P0.13), U5.14 (SDA)
- new net LCD_REFRESH: J2.4 (Pin_4), R8.2, TP2.1, U6.3 (~{INT}/SQW)
- new net QSPI_CS: U1.AD22 (TRACEDATA0/P1.00), U7.1 (~{CS})
- new net QSPI_D1: U1.AD20 (P0.24), U7.2 (DO(IO1))
- new net QSPI_D2: U1.AD18 (P0.22), U7.3 (IO2)
- no-connect marks 36 -> 33
Other:
- note added: "16MB flash"
- note added: "Fuel gauge"
- note added: "IMU"
- note added: "NRF52 has internal pullup for reset"
- note added: "Pimoroni: 500mah 37x30.5x5.3mm eBay: 500mah 35x30x5mm Amazon: 320mah 37x25.5x4.3mm"
- note added: "RTC"
- note added: "System can only be initially powered up off USB Microcontroller then latches battery power on Can shut down when battery empty to prevent overdischarge Bypass also included for developement purposes"
- note added: "~3.5V dropout 200mA max"
- note removed: "Also considering the BQ27220"
- note removed: "Battery fuel gauge"
- note removed: "Only 2mW dissipated"
- note removed: "~3.5V dropout 200mA max Wanted to use 1.8V but not sure how eink would react"
- moved on the sheet: C15, C34, C35, C36, C37, D2, J3, Q1, R7, R8, SW1, SW2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
