File: STM32WB55/Hardware/Hardware.kicad_sch (KiCad schematic)
At the start: 11 parts, among them J1 USB_C_Receptacle_USB2.0, J2 LCD, SW1 SW_Push, SW2 SW_Push, SW3 SW_Push, U1 STM32WB55CGUx

Commit message: Schematic progress
Parts:
- added C15, C34, C35: 1u, Capacitor_SMD:C_0402_1005Metric, symbol Device:C
- added D2: 1N5819WS, Diode_SMD:D_SOD-323, symbol Diode:1N5819WS
- added J2: BAT, local:Battery Pads, symbol Connector_Generic:Conn_01x02
- added Q1: AO3401A, Package_TO_SOT_SMD:SOT-23, symbol Transistor_FET:AO3401A
- added R8: 2K2, Resistor_SMD:R_0402_1005Metric, symbol Device:R
- added R8: 10K, Resistor_SMD:R_0402_1005Metric, symbol Device:R
- added U3: TP4054, Package_TO_SOT_SMD:SOT-23-5, symbol local:TP4054
- added U4: XC6206PxxxMR, Package_TO_SOT_SMD:SOT-23-3, symbol Regulator_Linear:XC6206PxxxMR
- added U7: W25Q128JVS, Package_SO:SOIC-8_5.23x5.23mm_P1.27mm, symbol Memory_Flash:W25Q128JVS
- added U?: LIS2DH12, Package_LGA:LGA-12_2x2mm_P0.5mm, symbol Sensor_Motion:LIS2DE12
- added U?: LIS3DH, Package_LGA:LGA-16_3x3mm_P0.5mm_LayoutBorder3x5y, symbol Sensor_Motion:LIS3DH
Connections:
- net +3V3: now also C35.1, U4.2 (VO), U7.8 (VCC)
- net GND: now also C15.2, C34.1, C35.2, J2.1 (Pin_1), R8.1, R8.1, U3.2 (GND), U4.1 (GND), U7.4 (GND)
- net VBUS: now also C15.1, D2.2 (A), Q1.1 (G), R8.2, U3.4 (VCC)
- new net: R8.2, U3.5 (PROG)
- new net: U?.6 (GND), U?.7 (GND), U?.8 (GND)
- new net: C34.2, D2.1 (K), Q1.2 (S), U4.3 (VI)
- new net: J2.2 (Pin_2), Q1.3 (D), U3.3 (BAT)
- new net: U?.10 (GND), U?.12 (GND), U?.5 (GND)
- new net QSPI_CS: U7.1 (~{CS})
- new net QSPI_D0: U7.5 (DI(IO0))
- new net QSPI_D1: U7.2 (DO(IO1))
- new net QSPI_D2: U7.3 (IO2)
- new net QSPI_D3: U7.7 (IO3)
- new net QSPI_SCK: U7.6 (CLK)
- no-connect marks 2 -> 3
Other:
- note added: "$0.4065"
- note added: "$0.4785"
- note added: "16MB flash"
- note added: "Battery charger 450mA charge current"
- note added: "Not much price differnce, ADCs could be handy"
- note added: "Pimoroni: 500mah 37x30.5x5.3mm eBay: 500mah 35x30x5mm Amazon: 320mah 37x25.5x4.3mm"
- note added: "Quite power hungry Lower capacities are less so"
- note added: "~3.5V dropout 200mA max output 1μA power consumption"
- moved on the sheet: U1

Commit message: Schematic progress
Parts:
- removed U?: LIS2DH12, Package_LGA:LGA-12_2x2mm_P0.5mm, symbol Sensor_Motion:LIS2DE12
- added C14: 470n, Capacitor_SMD:C_0402_1005Metric, symbol Device:C
- added C22: 10u, Capacitor_SMD:C_0402_1005Metric, symbol Device:C
- added C22: 1u, Capacitor_SMD:C_0402_1005Metric, symbol Device:C
- added J3: PROG, local:Program_Pads, symbol Connector_Generic:Conn_01x04
- added R6: R01 1%, Resistor_SMD:R_0805_2012Metric, symbol Device:R
- added R7 (x3): 10K, Resistor_SMD:R_0402_1005Metric, symbol Device:R
- added U2: BQ27441DRZR-G1A, Package_SON:Texas_S-PDSO-N12, symbol Battery_Management:BQ27441DRZR-G1A
- R8: value 2K2 -> 3.3K
Connections:
- net +3V3: now also U1.1 (VBAT), U1.20 (VDD), U1.35 (VDD), U?.1 (VDD_IO), U?.14 (VDD), U?.8 (CS), C22.1, C22.1, J3.4 (Pin_4), R7.1, R7.1
- net GND: now also U1.22 (VSSRF), U1.32 (VSSSMPS), U1.49 (VSS), U?.10 (GND), U?.12 (GND), U?.5 (GND), U?.7 (SDO/SA0), C14.2, C22.2, C22.2, J3.1 (Pin_1), R7.2, U2.13 (PAD), U2.3 (V_{SS})
- net USB_DN: now also U1.37 (PA11)
- net USB_DP: now also U1.38 (PA12)
- net VBUS: now also U1.40 (VDDUSB)
- net at U1.23 (VDDRF): now also U1.34 (VDDSMPS), U1.48 (VDD), U1.8 (VDDA)
- net SWDIO: now reaches U1.39 (PA13)
- net SWDIO: now also J3.3 (Pin_3)
- net SWDCLK: now reaches U1.41 (PA14)
- net SWDCLK: now also J3.2 (Pin_2)
- net +BATT: now reaches Q1.3 (D), U3.3 (BAT)
- net +BATT: now also R6.2, U2.7 (SRN); no longer J2.2 (Pin_2)
- net IMU_INT1: now reaches U?.11 (INT1)
- net IMU_INT1: now also U?.9 (INT2)
- net IMU_SCL: now reaches U?.4 (SCL/SPC)
- net IMU_SCL: now also R7.2
- net IMU_SDA: now reaches U?.6 (SDA/SDI/SDO)
- net IMU_SDA: now also R7.2
- new net: J2.2 (Pin_2), R6.1, U2.6 (BAT), U2.8 (SRP)
- new net: R7.1, U2.10 (BIN)
- new net: C14.1, U2.5 (V_{DD})
- new net FG_INT: U2.12 (GPOUT)
- new net FG_SCL: U2.2 (SCL)
- new net FG_SDA: U2.1 (SDA)
- no-connect marks 3 -> 6
Other:
- note added: "Battery charger 300mA charge current"
- note added: "Battery fuel gauge"
- note added: "Only 2mW dissipated"
- note removed: "$0.4065"
- note removed: "$0.4785"
- note removed: "Battery charger 450mA charge current"
- note removed: "Not much price differnce, ADCs could be handy"
- moved on the sheet: C15, C20, C21, C22, C34, C35, D2, J1, J2, Q1, R1, R2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

Commit message: Schematic progress
Parts:
- added AE?: Antenna_Chip, RF_Antenna:Johanson_2450AT43F0100, symbol Device:Antenna_Chip
- added C1, C2: 12p, Capacitor_SMD:C_0402_1005Metric, symbol Device:C
- added C22 (x7): 100nF, Capacitor_SMD:C_0402_1005Metric, symbol Device:C
- added C22 (x3): 4.7uF, Capacitor_SMD:C_0402_1005Metric, symbol Device:C
- added C22: 1uF, Capacitor_SMD:C_0402_1005Metric, symbol Device:C
- added C22: 10nF, Capacitor_SMD:C_0402_1005Metric, symbol Device:C
- added C3, C4: 6p8, Capacitor_SMD:C_0402_1005Metric, symbol Device:C
- added J6: FRONTLIGHT, symbol Connector_Generic:Conn_01x02
- added L1: 10uH, symbol Device:L
- added L2: 10nH, symbol Device:L
- added R7 (x3): 10K, Resistor_SMD:R_0402_1005Metric, symbol Device:R
- added R7: 100K, Resistor_SMD:R_0402_1005Metric, symbol Device:R
- added SW1: SW_Push, Button_Switch_SMD:Panasonic_EVQPUL_EVQPUC, symbol Switch:SW_Push
- added U?: MLPF-WB55-01E3, Package_CSP:WLCSP-6_1.4x1.0mm_P0.4mm, symbol Connector_Generic:Conn_01x06
- added Y1: 32MHz 8pF ±10ppm, Crystal:Crystal_SMD_2016-4Pin_2.0x1.6mm, symbol Device:Crystal_GND24
- added Y2: 32.768kHz 6pF ±20ppm, Crystal:Crystal_SMD_3215-2Pin_3.2x1.5mm, symbol Device:Crystal
- C14: value 470n -> 470nF; LCSC C47339 -> (none)
- C15, C21, C22, C34, C35: value 1u -> 1uF; LCSC C52923 -> (none)
- C20: value 100p -> 100nF; LCSC C52923 -> (none)
- C22: value 10u -> 10uF; LCSC C52923 -> (none)
- C22: value 1u -> 100nF; LCSC C52923 -> (none)
- U4: value XC6206PxxxMR -> XC6206P332MR
- gave numbers to parts that had none: 1
Connections:
- net +3V3: now also C22.1, C22.1, C22.1, C22.1, C22.1, C22.1, C22.1, C22.1, C22.1, R7.1, R7.1, R7.1, SW1.2
- net FG_SCL: now also R7.2
- net FG_SDA: now also R7.2
- net GND: now also C1.1, C2.2, C22.2, C22.2, C22.2, C22.2, C22.2, C22.2, C22.2, C22.2, C22.2, C22.2, C22.2, C22.2, C3.1, C4.2, R7.2, U?.1 (Pin_1), U?.2 (Pin_2), U?.3 (Pin_3), U?.4 (Pin_4), Y1.2, Y1.4
- net VBUS: now also C22.1
- net at U1.2 (PC14): now also C3.2, Y2.2
- net RF_OUT: now reaches U1.21 (RF1)
- net RF_OUT: now also U?.5 (Pin_5)
- net at U1.24 (OSC_OUT): now also C2.1, Y1.3
- net at U1.25 (OSC_IN): now also C1.2, Y1.1
- net at U1.3 (PC15): now also C4.1, Y2.1
- net at U1.31 (VFBSMPS): now also C22.1, L1.1
- net at U1.33 (VLXSMPS): now also L2.2
- net LIGHT_BUTTON: now reaches U1.4 (PH3)
- net LIGHT_BUTTON: now also R7.1, SW1.1
- net ~{RESET}: now reaches U1.7 (NRST)
- net ~{RESET}: now also C22.1, R7.2
- new net: L1.2, L2.1
- new net: AE?.1 (FEED), U?.6 (Pin_6)
- no-connect marks 6 -> 8
Other:
- note added: "11μA active 0.5μA sleep"
- note added: "16MB flash 10μA sleep >10mA read"
- note added: "3.3V LDO ~3.5V dropout but will still pass input voltage 200mA max output 1μA standby"
- note added: "Battery charger 300mA charge current 45μA shutdown"
- note added: "Battery fuel gauge 93μA active 21μA sleep 9μA hibernate 1μA shutdown"
- note added: "Considering moving to BQ27220 but no pre-existing KiCad symbols or Arduino libraries are available"
- note added: "Could switch to STM32WB5MM if certification required"
- note added: "Could this possibly be a 3.6V LDO instead?"
- note added: "LCD 15μA refresh 5mA frontlight"
- note added: "MCU 5.2mA tx 2.1μA stop 600nA standby 13nA shutdown"
- note added: "Near VDD & VBAT"
- note added: "Near VDDA"
- note added: "Near VDDSMPS"
- note added: "Near VDDUSB"
- note removed: "16MB flash"
- note removed: "Battery charger 300mA charge current"
- note removed: "Battery fuel gauge"
- note removed: "Quite power hungry Lower capacities are less so"
- note removed: "~3.5V dropout 200mA max output 1μA power consumption"
- moved on the sheet: C22, R7, SW1, SW2, SW3, U1

Commit message: Schematic progress and start PCB
Parts:
- removed AE?: Antenna_Chip, RF_Antenna:Johanson_2450AT43F0100, symbol Device:Antenna_Chip
- removed C1, C2: 12p, Capacitor_SMD:C_0402_1005Metric, symbol Device:C
- removed C22 (x6): 100nF, Capacitor_SMD:C_0402_1005Metric, symbol Device:C
- removed C22 (x3): 4.7uF, Capacitor_SMD:C_0402_1005Metric, symbol Device:C
- removed C22: 1uF, Capacitor_SMD:C_0402_1005Metric, symbol Device:C
- removed C22: 10nF, Capacitor_SMD:C_0402_1005Metric, symbol Device:C
- removed C3, C4: 6p8, Capacitor_SMD:C_0402_1005Metric, symbol Device:C
- removed J6: FRONTLIGHT, symbol Connector_Generic:Conn_01x02
- removed L1: 10uH, symbol Device:L
- removed L2: 10nH, symbol Device:L
- removed R7: 100K, Resistor_SMD:R_0402_1005Metric, symbol Device:R
- removed R7: 10K, Resistor_SMD:R_0402_1005Metric, symbol Device:R
- removed U1: STM32WB55CGUx, Package_DFN_QFN:QFN-48-1EP_7x7mm_P0.5mm_EP5.6x5.6mm, symbol MCU_ST_STM32WB:STM32WB55CGUx
- removed U7: W25Q128JVS, Package_SO:SOIC-8_5.23x5.23mm_P1.27mm, symbol Memory_Flash:W25Q128JVS
- removed U?: MLPF-WB55-01E3, Package_CSP:WLCSP-6_1.4x1.0mm_P0.4mm, symbol Connector_Generic:Conn_01x06
- removed Y1: 32MHz 8pF ±10ppm, Crystal:Crystal_SMD_2016-4Pin_2.0x1.6mm, symbol Device:Crystal_GND24
- removed Y2: 32.768kHz 6pF ±20ppm, Crystal:Crystal_SMD_3215-2Pin_3.2x1.5mm, symbol Device:Crystal
- added C20 (x3): 3.3pF, Capacitor_SMD:C_0402_1005Metric, symbol Device:C
- added D2, D3: LED, LED_SMD:LED_1206_3216Metric_ReverseMount_Hole1.8x2.4mm, symbol Device:LED
- added D2: 1N5819WS, Diode_SMD:D_SOD-323, symbol Diode:1N5819WS
- added J5: AUX, local:1x02_2.54_Pads, symbol Connector_Generic:Conn_01x02
- added Q2 (x2): AO3400A, Package_TO_SOT_SMD:SOT-23, symbol Transistor_FET:AO3400A
- added R7: 1K, Resistor_SMD:R_0402_1005Metric, symbol Device:R
- added R7: 470R, Resistor_SMD:R_0402_1005Metric, symbol Device:R
- added R8 (x2): 100K, Resistor_SMD:R_0402_1005Metric, symbol Device:R
- added R8: 10R, Resistor_SMD:R_0402_1005Metric, symbol Device:R
- added SW2: SW_Push, local:Panasonic_EVQPUL_EVQPUC, symbol Switch:SW_Push
- added U1: USBLC6-2SC6, Package_TO_SOT_SMD:SOT-23-6, symbol local:USBLC6-2SC6
- added U2: STM32WB5MMGH6TR, local:LCC-LGA-86_L11.0-W7.3_STM32WB5MMGH6TR, symbol local:STM32WB5MMGH6TR
- J1: LCSC (none) -> C3020046
- J2: footprint local:Battery Pads -> local:1x02_2.54_Pads
- J3: footprint local:Program_Pads -> local:1x04_2.54_Pads
- SW1, SW2, SW3: footprint Button_Switch_SMD:Panasonic_EVQPUL_EVQPUC -> local:Panasonic_EVQPUL_EVQPUC
- renumbered U4 to U5
Connections:
- net +3V3: now also D2.1 (K), J5.1 (Pin_1), R8.1, U2.15 (VBAT), U2.17 (VDDA), U2.4 (VREF+), U2.6 (VDDA)
- net GND: now also C20.2, C20.2, C20.2, Q2.2 (S), Q2.2 (S), R7.1, R8.2, R8.2, SW2.2, U1.2 (GND), U2., U2.16 (VSS), U2.31 (VSS), U2.5 (VSS), U2.57 (VSS), U2.58 (ANT_IN), U2.59 (RF_OUT), U2.60 (VSS), U2.72 (PE3), U2.73 (PD4), U2.83 (PC8), U2.84 (VSS), U2.86 (VSS)
- net IMU_INT1: no longer U5.9 (INT2)
- net LCD_REFRESH: now also U2.9 (PC1)
- net SWDCLK: now also U2.26 (PA14)
- net SWDIO: now also U2.25 (PA13)
- net USB_DN: now also U1.6 (I/O1), U2.30 (PA11); no longer J1.A7 (D-), J1.B7 (D-)
- net USB_DP: now also U1.4 (I/O2), U2.29 (PA12); no longer J1.A6 (D+), J1.B6 (D+)
- net VBUS: now also R7.1, U1.5 (VBUS)
- net DOWN_BUTTON renamed ~{SW_DOWN}
- net LIGHT_BUTTON renamed SW_LIGHT
- net SW_LIGHT: now also U2.13 (PH3-BOOT0)
- net MENU_BUTTON renamed ~{SW_MENU}
- net UP_BUTTON renamed ~{SW_UP}
- net ~{RESET} renamed ~{SW_RESET}
- net ~{SW_RESET}: now also SW2.1, U2.10 (NRST)
- new net: J1.A7 (D-), J1.B7 (D-), U1.1 (I/O1)
- new net: J1.A6 (D+), J1.B6 (D+), U1.3 (I/O2)
- new net: R7.2, R7.2, U2.32 (VDDUSB)
- new net: C20.1, U2.45 (PC5)
- new net: C20.1, U2.46 (PB11)
- new net: C20.1, U2.47 (PB10)
- new net: D2.2 (A), J5.2 (Pin_2), Q2.3 (D)
- new net: D2.1 (K), D3.1 (K), Q2.3 (D)
- new net: D2.2 (A), D3.2 (A), R8.2
- new net AUX_EN: Q2.1 (G), R8.1
- new net IMU_INT2: U5.9 (INT2)
- new net LIGHT_EN: Q2.1 (G), R8.1
- no-connect marks 8 -> 65
Other:
- note added: "USB"
- note removed: "16MB flash 10μA sleep >10mA read"
- note removed: "Could switch to STM32WB5MM if certification required"
- note removed: "Near VDD & VBAT"
- note removed: "Near VDDA"
- note removed: "Near VDDSMPS"
- note removed: "Near VDDUSB"
- moved on the sheet: C14, C15, C20, C21, C22, C34, C35, D2, J2, Q1, R1, R2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
