File: STM32WB55/Hardware/Hardware.kicad_pcb (KiCad board)
At the start: 2 copper layers, 13.6 x 6.9 mm, 11 parts, among them J1 USB_C_Receptacle_USB2.0, J2 LCD, SW1 SW_Push, SW2 SW_Push, SW3 SW_Push, U1 STM32WB55CGUx

Commit message: Schematic progress and start PCB
Parts:
- added C10: 1uF, Capacitor_SMD:C_0402_1005Metric, B.Cu at (133.6, 113.0)
- added C11: 100nF, Capacitor_SMD:C_0402_1005Metric, B.Cu at (133.6, 115.0)
- added C12: 10uF, Capacitor_SMD:C_0402_1005Metric, B.Cu at (133.6, 117.0)
- added C13: 1uF, Capacitor_SMD:C_0402_1005Metric, B.Cu at (133.6, 118.9)
- added C4: 3.3pF, Capacitor_SMD:C_0402_1005Metric, B.Cu at (136.5, 111.0)
- added C5: 470nF, Capacitor_SMD:C_0402_1005Metric, B.Cu at (136.5, 113.0)
- added C6: 1uF, Capacitor_SMD:C_0402_1005Metric, B.Cu at (136.5, 115.0)
- added C7: 100nF, Capacitor_SMD:C_0402_1005Metric, B.Cu at (136.5, 117.0)
- added C8: 1uF, Capacitor_SMD:C_0402_1005Metric, B.Cu at (136.5, 118.9)
- added C9: 1uF, Capacitor_SMD:C_0402_1005Metric, B.Cu at (133.6, 111.0)
- added D1: 1N5819WS, Diode_SMD:D_SOD-323, B.Cu at (135.8, 121.4)
- added D2: LED, LED_SMD:LED_1206_3216Metric_ReverseMount_Hole1.8x2.4mm, B.Cu at (105.0, 104.5)
- added D3: LED, LED_SMD:LED_1206_3216Metric_ReverseMount_Hole1.8x2.4mm, B.Cu at (121.5, 104.5)
- added D4: 1N5819WS, Diode_SMD:D_SOD-323, B.Cu at (114.6, 127.0)
- added J3: BAT, local:1x02_2.54_Pads, B.Cu at (134.1, 106.2)
- added J4: LCD, Connector_FFC-FPC:Molex_54548-1071_1x10-1MP_P0.5mm_Horizontal, B.Cu at (113.2, 79.4)
- added J5: AUX, local:1x02_2.54_Pads, B.Cu at (118.6, 125.1)
- added Q1: AO3401A, Package_TO_SOT_SMD:SOT-23, B.Cu at (140.4, 112.3)
- added Q2: AO3400A, Package_TO_SOT_SMD:SOT-23, B.Cu at (159.8, 121.6)
- added Q3: AO3400A, Package_TO_SOT_SMD:SOT-23, B.Cu at (124.5, 132.0)
- added R10: 10K, Resistor_SMD:R_0402_1005Metric, B.Cu at (144.3, 111.1)
- added R11: 10R, Resistor_SMD:R_0402_1005Metric, B.Cu at (160.8, 124.9)
- added R12: 100K, Resistor_SMD:R_0402_1005Metric, B.Cu at (144.3, 113.0)
- added R13: 10K, Resistor_SMD:R_0402_1005Metric, B.Cu at (144.3, 115.0)
- added R14: 10K, Resistor_SMD:R_0402_1005Metric, B.Cu at (115.3, 129.5)
- added R15: 100K, Resistor_SMD:R_0402_1005Metric, B.Cu at (125.5, 135.2)
- added R3: R01 1%, Resistor_SMD:R_0805_2012Metric, B.Cu at (131.4, 126.1)
- added R4: 470R, Resistor_SMD:R_0402_1005Metric, B.Cu at (147.2, 111.1)
- added R5: 1K, Resistor_SMD:R_0402_1005Metric, B.Cu at (147.2, 113.0)
- added R6: 10K, Resistor_SMD:R_0402_1005Metric, B.Cu at (147.2, 115.0)
- added R7: 10K, Resistor_SMD:R_0402_1005Metric, B.Cu at (147.2, 117.0)
- added R8: 10K, Resistor_SMD:R_0402_1005Metric, B.Cu at (147.2, 119.0)
- added R9: 3.3K, Resistor_SMD:R_0402_1005Metric, B.Cu at (147.2, 121.0)
- added SW4: SW_Push, local:Panasonic_EVQPUL_EVQPUC, B.Cu at (126.2, 87.0)
- added SW5: SW_Push, local:Panasonic_EVQPUL_EVQPUC, B.Cu at (126.2, 98.0)
- added U2: STM32WB5MMGH6TR, local:LCC-LGA-86_L11.0-W7.3_STM32WB5MMGH6TR, B.Cu at (113.2, 100.3)
- added U3: BQ27441DRZR-G1A, Package_SON:Texas_S-PDSO-N12, B.Cu at (130.5, 122.3)
- added U4: TP4054, Package_TO_SOT_SMD:SOT-23-5, B.Cu at (129.6, 112.3)
- added U5: LIS3DH, Package_LGA:LGA-16_3x3mm_P0.5mm_LayoutBorder3x5y, B.Cu at (140.6, 125.7)
- added U6: XC6206P332MR, Package_TO_SOT_SMD:SOT-23-3, B.Cu at (129.6, 116.7)
- C1: value 100p -> 100nF; moved to B.Cu
- C2, C3: value 1u -> 3.3pF; moved to B.Cu
- J1, R1, R2: moved to B.Cu
- J2: value LCD -> PROG; footprint Connector_FFC-FPC:Molex_54548-1071_1x10-1MP_P0.5mm_Horizontal -> local:1x04_2.54_Pads; moved to B.Cu
- SW1, SW2, SW3: footprint Button_Switch_SMD:Panasonic_EVQPUL_EVQPUC -> local:Panasonic_EVQPUL_EVQPUC; moved to B.Cu
- U1: value STM32WB55CGUx -> USBLC6-2SC6; footprint Package_DFN_QFN:QFN-48-1EP_7x7mm_P0.5mm_EP5.6x5.6mm -> Package_TO_SOT_SMD:SOT-23-6; moved to B.Cu
- moved J2 62.5 mm to (109.7, 111.0), turned to -90 degrees
- moved U1 52.6 mm to (175.3, 72.4), turned to 180 degrees
- moved SW2 50.2 mm to (100.2, 98.0), turned to -90 degrees
- moved SW1 46.3 mm to (100.2, 76.0), turned to -90 degrees
- moved SW3 21.9 mm to (126.2, 76.0), turned to 90 degrees
- moved J1 18.8 mm to (103.8, 87.0), turned to 90 degrees
- moved R1 12.3 mm to (142.9, 76.1), turned to 180 degrees
- moved R2 12.3 mm to (142.9, 78.1), turned to 180 degrees
- moved C1 6.49 mm to (145.7, 76.1), turned to 180 degrees
- moved C2 6.49 mm to (145.7, 78.1), turned to 180 degrees
- moved C3 6.49 mm to (145.7, 80.1), turned to 180 degrees
Connections:
- net /DOWN_BUTTON renamed /~{SW_UP}
- C1 pad 1: +3V3 -> /~{SW_RESET}
- C2 pad 1: +3V3 -> Net-(U2-PC5)
- C3 pad 1: +3V3 -> Net-(U2-PB11)
- J1 pad A6: /USB_DP -> Net-(J1-D+-PadA6)
- J1 pad A7: /USB_DN -> Net-(J1-D--PadA7)
- J1 pad B6: /USB_DP -> Net-(J1-D+-PadA6)
- J1 pad B7: /USB_DN -> Net-(J1-D--PadA7)
- J2 pad 1: /LCD_SCLK -> GND
- J2 pad 2: /LCD_SDI -> /SWDCLK
- J2 pad 3: /LCD_CS -> /SWDIO
- J2 pad 4: /LCD_REFRESH -> +3V3
- SW1 pad 1: /UP_BUTTON -> /SW_LIGHT
- SW1 pad 2: GND -> +3V3
- SW2 pad 1: /MENU_BUTTON -> /~{SW_RESET}
- U1 pad 1: unconnected-(U1-VBAT-Pad1) -> Net-(J1-D--PadA7)
- U1 pad 2: unconnected-(U1-PC14-Pad2) -> GND
- U1 pad 3: unconnected-(U1-PC15-Pad3) -> Net-(J1-D+-PadA6)
- U1 pad 4: unconnected-(U1-PH3-Pad4) -> /USB_DP
- U1 pad 5: unconnected-(U1-PB8-Pad5) -> VBUS
- U1 pad 6: unconnected-(U1-PB9-Pad6) -> /USB_DN
Other:
- board size 13.6 x 6.9 mm -> 52.8 x 38 mm
- board text added: "08/2024"
- board text added: "@edatki"
- board text added: "DN"
- board text added: "LED"
- board text added: "OK"
- board text added: "QUECTOWATCH"
- board text added: "RES"
- board text added: "UP"

Commit message: Ordered
Parts:
- removed D2, D3: LED, LED_SMD:LED_1206_3216Metric_ReverseMount_Hole1.8x2.4mm
- removed R11: 10R, Resistor_SMD:R_0402_1005Metric
- added J6: LED+, TestPoint:TestPoint_Pad_2.0x2.0mm, F.Cu at (103.0, 104.5)
- added J7: LED-, TestPoint:TestPoint_Pad_2.0x2.0mm, F.Cu at (123.5, 104.5)
- added JP1: Jumper_2_Open, Jumper:SolderJumper-2_P1.3mm_Open_TrianglePad1.0x1.5mm, B.Cu at (104.8, 99.0)
- SW1, SW2, SW3, SW4, SW5: footprint local:Panasonic_EVQPUL_EVQPUC -> local:Panasonic_EVQPUA_EVQPUJ
- moved U1 68.6 mm to (108.5, 88.2), turned to 0 degrees
- moved R6 57.0 mm to (104.5, 77.2)
- moved R15 56.5 mm to (120.2, 79.0), turned to -90 degrees
- moved Q3 56.3 mm to (121.5, 75.8), turned to -90 degrees
- moved U3 54.6 mm to (105.2, 73.9), turned to -90 degrees
- moved R3 53.9 mm to (105.2, 79.0), turned to 0 degrees
- moved C5 52.6 mm to (105.5, 70.5)
- moved D1 50.6 mm to (105.2, 81.0)
- moved R9 50.2 mm to (111.2, 86.0), turned to 0 degrees
- moved J3 49.1 mm to (101.0, 70.0), turned to -90 degrees
- moved D4 46.5 mm to (124.2, 81.5), turned to 90 degrees
- moved J2 45.1 mm to (127.9, 69.8), turned to 90 degrees
- moved C1 44.8 mm to (107.2, 99.0), turned to -90 degrees
- moved U5 44.6 mm to (111.2, 92.0)
- moved J5 44.2 mm to (122.0, 81.0), turned to 0 degrees
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Connections:
- C1 pad 1: /~{SW_RESET} -> Net-(JP1-B)
- U2 pad 10: /~{SW_RESET} -> Net-(JP1-B)
- U2 pad 11: unconnected-(U2-PB9-Pad11) -> /~{SW_RESET}
- U2 pad 12: unconnected-(U2-PC0-Pad12) -> /IMU_INT2
- U2 pad 14: unconnected-(U2-PB8-Pad14) -> /IMU_INT1
- U2 pad 18: unconnected-(U2-PB7-Pad18) -> /IMU_SDA
- U2 pad 19: unconnected-(U2-PB5-Pad19) -> /LCD_SDI
- U2 pad 21: unconnected-(U2-PB3-Pad21) -> /LCD_SCLK
- U2 pad 22: unconnected-(U2-PC10-Pad22) -> GND
- U2 pad 23: unconnected-(U2-PC11-Pad23) -> GND
- U2 pad 24: unconnected-(U2-PC12-Pad24) -> GND
- U2 pad 27: unconnected-(U2-PA15-Pad27) -> /LCD_CS
- U2 pad 37: unconnected-(U2-PB14-Pad37) -> /~{SW_UP}
- U2 pad 38: unconnected-(U2-PB15-Pad38) -> /~{SW_MENU}
- U2 pad 39: unconnected-(U2-PB6-Pad39) -> /~{SW_DOWN}
- U2 pad 40: unconnected-(U2-PC13-Pad40) -> /LCD_REFRESH
- U2 pad 41: unconnected-(U2-PB12-Pad41) -> GND
- U2 pad 42: unconnected-(U2-PE4-Pad42) -> GND
- U2 pad 48: unconnected-(U2-PB2-Pad48) -> /LIGHT_EN
- U2 pad 49: unconnected-(U2-PC4-Pad49) -> GND
- U2 pad 50: unconnected-(U2-PA8-Pad50) -> GND
- U2 pad 51: unconnected-(U2-PA9-Pad51) -> /IMU_SCL
- U2 pad 52: unconnected-(U2-PA7-Pad52) -> /FG_SCL
- U2 pad 56: unconnected-(U2-PA3-Pad56) -> /AUX_EN
- U2 pad 63: unconnected-(U2-PD14-Pad63) -> GND
- U2 pad 64: unconnected-(U2-PE1-Pad64) -> GND
- U2 pad 65: unconnected-(U2-PD13-Pad65) -> GND
- U2 pad 66: unconnected-(U2-PD12-Pad66) -> GND
- U2 pad 67: unconnected-(U2-PD7-Pad67) -> GND
- U2 pad 68: unconnected-(U2-PD2-Pad68) -> GND
- U2 pad 69: unconnected-(U2-PC9-Pad69) -> GND
- U2 pad 70: unconnected-(U2-PD3-Pad70) -> GND
- U2 pad 71: unconnected-(U2-PC7-Pad71) -> GND
- U2 pad 74: unconnected-(U2-PD9-Pad74) -> GND
- U2 pad 75: unconnected-(U2-PD8-Pad75) -> GND
- U2 pad 76: unconnected-(U2-PD15-Pad76) -> GND
- U2 pad 77: unconnected-(U2-PD10-Pad77) -> GND
- U2 pad 78: unconnected-(U2-PE2-Pad78) -> GND
- U2 pad 79: unconnected-(U2-PE0-Pad79) -> GND
- U2 pad 8: unconnected-(U2-PC2-Pad8) -> /FG_INT
- U2 pad 80: unconnected-(U2-PD5-Pad80) -> GND
- U2 pad 81: unconnected-(U2-PD6-Pad81) -> GND
- U2 pad 82: unconnected-(U2-PD11-Pad82) -> GND
- U2 pad 9: /LCD_REFRESH -> /FG_SDA
Routing:
- net +3V3: track 0.00 -> 88.7 mm, vias 0 -> 4
- net VBUS: track 0.00 -> 52.4 mm, vias 0 -> 4
- net /AUX_EN: track 0.00 -> 44.8 mm, vias 0 -> 4
- net /FG_SCL: track 0.00 -> 44.3 mm, vias 0 -> 3
- net /SWDIO: track 0.00 -> 38.1 mm, vias 0 -> 2
- net /SWDCLK: track 0.00 -> 37.0 mm, vias 0 -> 2
- net /FG_SDA: track 0.00 -> 36.4 mm, vias 0 -> 2
- net /USB_DP: track 0.00 -> 35.6 mm, vias 0 -> 2
- net /SW_LIGHT: track 0.00 -> 33.1 mm, vias 0 -> 2
- net /USB_DN: track 0.00 -> 32.0 mm, vias 0 -> 2
- net /~{SW_UP}: track 0.00 -> 31.6 mm
- net GND: track 0.00 -> 28.9 mm, vias 0 -> 230
- net /FG_INT: track 0.00 -> 28.5 mm, vias 0 -> 2
- net Net-(#FLG03-pwr): track 0.00 -> 21.3 mm
- net /LCD_REFRESH: track 0.00 -> 20.9 mm, vias 0 -> 2
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- added copper zone on B.Cu, net GND
- added copper zone on F.Cu, net GND
Other:
- board size 52.8 x 38 mm -> 32 x 38 mm
- board text added: "3V3"
- board text added: "BACK"
- board text added: "CLK"
- board text added: "DOWN"
- board text added: "ENTER"
- board text added: "GND"
- board text added: "IO"
- board text added: "LIGHT"
- board text added: "REV 3.0 16/08/2024"
- board text removed: "DN"
- board text removed: "LED"
- board text removed: "OK"
- board text removed: "RES"
